File: Hardware/Amplified-Mic-Electret.brd (EAGLE design)
At the start: 16.5 x 10.2 mm, 18 parts, among them M1 MIC9.7MM, U1 OPA344

Commit message: Midway changes
Parts:
- moved LOGO1 1.27 mm to (3.81, 1.27)
- moved C4 0.90 mm to (5.84, 3.17)
Changed lines of the file:
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@@
 <setting verticaltext="up"/>
 </settings>
-<grid distance="0.025" unitdist="inch" unit="inch" style="lines" multiple="1" display="yes" altdistance="0.005" altunitdist="inch" altunit="inch"/>
+<grid distance="0.05" unitdist="inch" unit="inch" style="lines" multiple="1" display="yes" altdistance="0.005" altunitdist="inch" altunit="inch"/>
 <layers>
 <layer number="1" name="Top" color="4" fill="1" visible="yes" active="yes"/>
@@
 <layer number="101" name="Patch_Top" color="12" fill="4" visible="no" active="yes"/>
 <layer number="102" name="Vscore" color="7" fill="1" visible="no" active="yes"/>
-<layer number="103" name="tMap" color="7" fill="1" visible="yes" active="yes"/>
+<layer number="103" name="tMap" color="7" fill="1" visible="no" active="yes"/>
 <layer number="104" name="Name" color="7" fill="1" visible="no" active="yes"/>
-<layer number="105" name="tPlate" color="7" fill="1" visible="yes" active="yes"/>
-<layer number="106" name="bPlate" color="7" fill="1" visible="yes" active="yes"/>
-<layer number="107" name="Crop" color="7" fill="1" visible="yes" active="yes"/>
+<layer number="105" name="tPlate" color="7" fill="1" visible="no" active="yes"/>
+<layer number="106" name="bPlate" color="7" fill="1" visible="no" active="yes"/>
+<layer number="107" name="Crop" color="7" fill="1" visible="no" active="yes"/>
 <layer number="116" name="Patch_BOT" color="9" fill="4" visible="no" active="yes"/>
 <layer number="121" name="_tsilk" color="7" fill="1" visible="no" active="yes"/>
 <layer number="122" name="_bsilk" color="7" fill="1" visible="no" active="yes"/>
-<layer number="125" name="_tNames" color="7" fill="1" visible="yes" active="yes"/>
-<layer number="144" name="Drill_legend" color="7" fill="1" visible="yes" active="yes"/>
+<layer number="125" name="_tNames" color="7" fill="1" visible="no" active="yes"/>
+<layer number="144" name="Drill_legend" color="7" fill="1" visible="no" active="yes"/>
 <layer number="151" name="HeatSink" color="7" fill="1" visible="no" active="yes"/>
-<layer number="199" name="Contour" color="7" fill="1" visible="yes" active="yes"/>
+<layer number="199" name="Contour" color="7" fill="1" visible="no" active="yes"/>
 <layer number="200" name="200bmp" color="1" fill="10" visible="no" active="no"/>
 <layer number="201" name="201bmp" color="2" fill="1" visible="no" active="no"/>
@@
 <layer number="207" name="207bmp" color="8" fill="10" visible="no" active="yes"/>
 <layer number="208" name="208bmp" color="9" fill="10" visible="no" active="yes"/>
-<layer number="209" name="209bmp" color="7" fill="1" visible="yes" active="yes"/>
-<layer number="210" name="210bmp" color="7" fill="1" visible="yes" active="yes"/>
-<layer number="211" name="211bmp" color="7" fill="1" visible="yes" active="yes"/>
-<layer number="212" name="212bmp" color="7" fill="1" visible="yes" active="yes"/>
-<layer number="213" name="213bmp" color="7" fill="1" visible="yes" active="yes"/>
-<layer number="214" name="214bmp" color="7" fill="1" visible="yes" active="yes"/>
-<layer number="215" name="215bmp" color="7" fill="1" visible="yes" active="yes"/>
-<layer number="216" name="216bmp" color="7" fill="1" visible="yes" active="yes"/>
+<layer number="209" name="209bmp" color="7" fill="1" visible="no" active="yes"/>
+<layer number="210" name="210bmp" color="7" fill="1" visible="no" active="yes"/>
+<layer number="211" name="211bmp" color="7" fill="1" visible="no" active="yes"/>
+<layer number="212" name="212bmp" color="7" fill="1" visible="no" active="yes"/>
+<layer number="213" name="213bmp" color="7" fill="1" visible="no" active="yes"/>
+<layer number="214" name="214bmp" color="7" fill="1" visible="no" active="yes"/>
+<layer number="215" name="215bmp" color="7" fill="1" visible="no" active="yes"/>
+<layer number="216" name="216bmp" color="7" fill="1" visible="no" active="yes"/>
 <layer number="217" name="217bmp" color="18" fill="1" visible="no" active="no"/>
 <layer number="218" name="218bmp" color="19" fill="1" visible="no" active="no"/>
@@
 <attribute name="PROD_ID" value="CAP-09137" x="8.89" y="8.89" size="1.778" layer="27" display="off"/>
 </element>
-<element name="C4" library="SparkFun-Capacitors" package="0603-CAP" value="0.1uF" x="5.207" y="3.81" smashed="yes">
-<attribute name="NAME" x="4.318" y="4.5085" size="0.4064" layer="25"/>
-<attribute name="VALUE" value="0.1uF" x="4.5085" y="2.794" size="0.4064" layer="27"/>
-<attribute name="PROD_ID" value="CAP-00810" x="5.207" y="3.81" size="1.778" layer="27" display="off"/>
+<element name="C4" library="SparkFun-Capacitors" package="0603-CAP" value="0.1uF" x="5.842" y="3.175" smashed="yes">
+<attribute name="NAME" x="4.953" y="3.8735" size="0.4064" layer="25"/>
+<attribute name="VALUE" value="0.1uF" x="5.1435" y="2.159" size="0.4064" layer="27"/>
+<attribute name="PROD_ID" value="CAP-00810" x="5.842" y="3.175" size="1.778" layer="27" display="off"/>
 </element>
 <element name="JP2" library="SparkFun" package="FIDUCIAL-1X2" value="FIDUCIAL1X2" x="12.8524" y="9.0932"/>
@@
 <element name="FRAME1" library="SparkFun-Aesthetics" package="CREATIVE_COMMONS" value="FRAME-LETTER" x="-11.70645625" y="-8.89"/>
 <element name="U$2" library="SparkFun-Aesthetics" package="REVISION" value="REVISION" x="0" y="-11.43"/>
-<element name="LOGO1" library="SparkFun-Aesthetics" package="OSHW-LOGO-S" value="OSHW-LOGOS" x="5.08" y="1.27"/>
+<element name="LOGO1" library="SparkFun-Aesthetics" package="OSHW-LOGO-S" value="OSHW-LOGOS" x="3.81" y="1.27"/>
 </elements>
 <signals>
@@
 <vertex x="16.51" y="0"/>
 </polygon>
-<wire x1="3.08" y1="6.35" x2="4.357" y2="3.81" width="0" layer="19" extent="1-1"/>
 </signal>
 <signal name="VCC">
@@
 <wire x1="8.255" y1="2.54" x2="8.255" y2="1.905" width="0.254" layer="1"/>
 <wire x1="4.953" y1="5.5" x2="5.207" y2="5.573" width="0.254" layer="1"/>
-<wire x1="5.715" y1="3.81" x2="5.715" y2="4.318" width="0.254" layer="1"/>
 <wire x1="4.953" y1="5.5" x2="5.08" y2="5.715" width="0.254" layer="1"/>
-<wire x1="5.715" y1="4.318" x2="4.953" y2="5.08" width="0.254" layer="1"/>
-<wire x1="4.953" y1="5.08" x2="4.953" y2="5.5" width="0.254" layer="1"/>
 <wire x1="6.67" y1="4.13" x2="7.5899" y2="4.13" width="0.254" layer="1"/>
-<wire x1="6.35" y1="3.81" x2="6.67" y2="4.13" width="0.254" layer="1"/>
-<wire x1="6.057" y1="3.81" x2="5.715" y2="3.81" width="0.254" layer="1"/>
-<wire x1="5.715" y1="3.81" x2="6.35" y2="3.81" width="0.254" layer="1"/>
 <wire x1="8.255" y1="2.54" x2="8.04" y2="2.54" width="0.254" layer="1"/>
 <wire x1="7.5899" y1="4.13" x2="7.5899" y2="3.2051" width="0.254" layer="1"/>
 <wire x1="7.5899" y1="3.2051" x2="8.255" y2="2.54" width="0.254" layer="1"/>
+<wire x1="4.953" y1="5.5" x2="4.953" y2="5.207" width="0.254" layer="1"/>
+<wire x1="4.953" y1="5.207" x2="6.35" y2="3.81" width="0.254" layer="1"/>
+<wire x1="6.35" y1="3.81" x2="6.35" y2="3.517" width="0.254" layer="1"/>
+<wire x1="6.35" y1="3.517" x2="6.692" y2="3.175" width="0.254" layer="1"/>
+<wire x1="6.67" y1="4.13" x2="6.35" y2="3.81" width="0.254" layer="1"/>
 </signal>
 <signal name="N$2">
