File: Hardware/SparkFun_Amplified-Mic-v13.brd (EAGLE design)
At the start: 16.5 x 10.2 mm, 16 parts, among them M1 MIC9.7MM, U1 OPA344

Commit message: few changes made
Parts:
- removed FRAME1: FRAME-LETTER, SparkFun-Aesthetics:CREATIVE_COMMONS
- C1: value 0.1uF -> 4.7u; device SparkFun:0402-CAP -> rcl:C0603
- C2: value 1uF -> 1.5u; device SparkFun:0402-CAP -> rcl:C0603
- C3: value 100pF -> .1p; device SparkFun:0402-CAP -> rcl:C0603
- R1: device SparkFun:0402-RES -> rcl:R0603
- R4: value 1K -> 5k; device SparkFun:0402-RES -> rcl:R0603
- R5: value 100K -> 800k; device SparkFun:0402-RES -> rcl:R0603
- moved U$1 18.0 mm to (25.9, -1.91)
- moved R1 0.76 mm to (4.19, 6.35)
Routing:
- net N$1: track 9.94 -> 12.1 mm
- net VCC: track 15.1 -> 16.7 mm
- net N$2: track 4.67 -> 5.27 mm
Other:
- board size 16.5 x 10.2 mm -> 20.6 x 10.2 mm
