File: Hardware/SparkFun_Amplified-Mic.sch (EAGLE design)
At the start: 17 parts, among them M1 MIC9.7MM, U1 OPA344

Commit message: Updated Board and Schematic files. Added product ID to Res5 and removed 10mils of board
Parts:
- R5: device SparkFun-Resistors:2.2MOHM-1/10W-5%(0603) -> SparkFun-Resistors:820KOHM-1/10W-1%(0603)
Changed lines of the file:
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@@
 <setting verticaltext="up"/>
 </settings>
-<grid distance="0.1" unitdist="inch" unit="inch" style="lines" multiple="1" display="yes" altdistance="0.01" altunitdist="inch" altunit="inch"/>
+<grid distance="0.1" unitdist="inch" unit="inch" style="lines" multiple="1" display="no" altdistance="0.01" altunitdist="inch" altunit="inch"/>
 <layers>
 <layer number="1" name="Top" color="4" fill="1" visible="no" active="no"/>
@@
 <layer number="255" name="routoute" color="7" fill="1" visible="yes" active="yes"/>
 </layers>
-<schematic>
+<schematic xreflabel="%F%N/%S" xrefpart="/%S.%C%R">
 <attributes>
 </attributes>
@@
 <part name="R3" library="SparkFun-Resistors" deviceset="10KOHM-1/10W-1%(0603)" device="0603" value="10K"/>
 <part name="R4" library="SparkFun-Resistors" deviceset="10KOHM-1/10W-1%(0603)" device="0603" value="10K"/>
-<part name="R5" library="SparkFun-Resistors" deviceset="2.2MOHM-1/10W-5%(0603)" device="" value="820k"/>
+<part name="R5" library="SparkFun-Resistors" deviceset="820KOHM-1/10W-1%(0603)" device="" value="820k"/>
 <part name="C2" library="SparkFun-Capacitors" deviceset="4.7UF-6.3V-10%(0603)" device="0603" value="4.7uF"/>
 <part name="C4" library="SparkFun-Capacitors" deviceset="0.1UF-25V(+80/-20%)(0603)" device="" value="0.1uF"/>
