File: Hardware/Electret_Microphone_Breakout.brd (EAGLE design)
At the start: 20.3 x 10.2 mm, 17 parts, among them U1 OPA344

Commit message: Updated Board Files
Parts:
- moved JP3 0.36 mm to (1.02, 1.02)
